File: Skayboard/Skayboard.kicad_pcb (KiCad board)
At the start: 2 copper layers, 354.9 x 107.3 mm, 237 parts, among them J1 D+, J2 D-, SW1 C3 Tangerine, SW10 C3 Tangerine, SW11 C3 Tangerine, SW12 C3 Tangerine, SW13 C3 Tangerine, SW14 C3 Tangerine, SW15 C3 Tangerine, SW16 C3 Tangerine, SW17 C3 Tangerine, SW18 C3 Tangerine, SW19 C3 Tangerine, SW2 C3 Tangerine, SW20 C3 Tangerine, SW21 C3 Tangerine, SW22 C3 Tangerine, SW23 C3 Tangerine, SW24 C3 Tangerine, SW25 C3 Tangerine, SW26 C3 Tangerine, SW27 C3 Tangerine, SW28 C3 Tangerine, SW29 C3 Tangerine, SW3 C3 Tangerine, SW30 C3 Tangerine, SW31 C3 Tangerine, SW32 C3 Tangerine, SW33 C3 Tangerine, SW34 C3 Tangerine, SW35 C3 Tangerine, SW36 C3 Tangerine, SW37 RST, SW38 C3 Tangerine, SW39 C3 Tangerine, SW4 C3 Tangerine, SW40 C3 Tangerine, SW41 C3 Tangerine, SW42 C3 Tangerine, SW43 C3 Tangerine, SW44 C3 Tangerine, SW45 C3 Tangerine, SW46 C3 Tangerine, SW47 C3 Tangerine, SW48 C3 Tangerine, SW49 C3 Tangerine, SW5 C3 Tangerine, SW50 C3 Tangerine, SW51 C3 Tangerine, SW52 C3 Tangerine, SW53 C3 Tangerine, SW54 C3 Tangerine, SW55 C3 Tangerine, SW56 C3 Tangerine, SW57 C3 Tangerine, SW58 C3 Tangerine, SW59 C3 Tangerine, SW6 C3 Tangerine, SW60 C3 Tangerine, SW61 C3 Tangerine, SW62 C3 Tangerine, SW63 C3 Tangerine, SW64 C3 Tangerine, SW65 C3 Tangerine, SW66 C3 Tangerine, SW67 C3 Tangerine, SW68 C3 Tangerine, SW69 C3 Tangerine, SW7 C3 Tangerine, SW70 C3 Tangerine, SW71 C3 Tangerine, SW72 C3 Tangerine, SW73 C3 Tangerine, SW74 C3 Tangerine, SW75 C3 Tangerine, SW76 C3 Tangerine, SW77 C3 Tangerine, SW8 C3 Tangerine, SW9 C3 Tangerine, U1 ATmega32U4-AU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

Commit message: Diodes placed, first row of LEDs almost done
Parts:
- added REF**: Stabilizer_Cherry_MX_2u, Mounting_Keyboard_Stabilizer:Stabilizer_Cherry_MX_2u, F.Cu at (404.9, 248.6)
- added REF**: Stabilizer_Cherry_MX_2u, Mounting_Keyboard_Stabilizer:Stabilizer_Cherry_MX_2u, F.Cu at (409.7, 229.5)
- added REF**: Stabilizer_Cherry_MX_2u, Mounting_Keyboard_Stabilizer:Stabilizer_Cherry_MX_2u, F.Cu at (412.0, 191.4)
- added REF**: Stabilizer_Cherry_MX_2u, Mounting_Keyboard_Stabilizer:Stabilizer_Cherry_MX_2u, F.Cu at (166.8, 248.6)
- added REF**: Stabilizer_Cherry_MX_6.25u, Mounting_Keyboard_Stabilizer:Stabilizer_Cherry_MX_6.25u, F.Cu at (276.3, 267.6)
- D100, D101, D102, D103, D104, D105, D106, D107, D108, D109, D110, D111, D112, D113, D114, D115, D116, D117, D118, D119, D12, D120, D121, D122, D123, D124, D125, D126, D127, D128, D129, D13, D130, D131, D132, D133, D134, D135, D136, D137, D138, D139, D14, D140, D141, D142, D143, D144, D145, D146, D147, D148, D149, D150, D151, D152, D20, D21, D22, D23, D24, D25, D26, D27, D32, D33, D34, D35, D36, D37, D38, D39, D40, D41, D42, D43, D44, D45, D46, D47, D48, D49, D50, D51, D52, D53, D54, D55, D56, D57, D58, D59, D60, D61, D62, D63, D64, D65, D66, D67, D68, D69, D70, D71, D72, D73, D74, D75, D76, D77, D78, D79, D80, D81, D82, D83, D84, D85, D86, D87, D88, D89, D90, D91, D92, D93, D94, D95, D96, D97, D98, D99: moved to B.Cu
- moved D24 366.0 mm to (192.9, 196.7), turned to 180 degrees
- moved D32 356.5 mm to (212.0, 196.7), turned to 180 degrees
- moved D48 331.7 mm to (283.9, 263.1), turned to 270 degrees
- moved D49 327.7 mm to (250.1, 196.7), turned to 180 degrees
- moved D45 293.1 mm to (267.1, 205.8), turned to 270 degrees
- moved D46 279.7 mm to (272.0, 224.9), turned to 270 degrees
- moved D37 279.4 mm to (248.0, 205.8), turned to 270 degrees
- moved D36 270.9 mm to (238.8, 186.8), turned to 270 degrees
- moved D61 256.1 mm to (285.6, 196.7), turned to 180 degrees
- moved D39 255.4 mm to (262.4, 244.0), turned to 270 degrees
- moved D40 247.5 mm to (231.1, 196.7), turned to 180 degrees
- moved D38 245.0 mm to (253.0, 224.8), turned to 270 degrees
- moved D53 237.1 mm to (266.6, 196.7), turned to 180 degrees
- moved D138 233.9 mm to (448.1, 263.1), turned to 270 degrees
- moved D73 233.5 mm to (326.3, 196.7), turned to 180 degrees
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Connections:
- D11 pad 1: (no net) -> +5V
- D11 pad 2: (no net) -> Net-(D11-Pad2)
- D11 pad 3: (no net) -> GND
- D11 pad 4: (no net) -> DIN
Other:
- outline, holes or cut-outs redrawn
