File: kicad/inc/LED.kicad_sch (KiCad schematic)
At the start: 2 parts

Commit message: feat: finishes schematic, starts work on PCB
Parts:
- LED1: footprint LED_SK6812MINI-E -> Skayboard:SK6812MINI-E
- renumbered C1 to C7
Connections:
- net DIN: now also LED1.4 (DIN); no longer LED1.3 (DIN)
- net DOUT: now also LED1.2 (DOUT); no longer LED1.1 (DOUT)
- net GND: now also LED1.3 (VSS); no longer LED1.2 (VSS)
- net VCC: now also LED1.1 (VDD); no longer LED1.4 (VDD)
Changed lines of the file:
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@@
   (symbol (lib_id "power:VCC") (at 63.5 24.13 0) (unit 1)
     (in_bom yes) (on_board yes)
-    (property "Reference" "#PWR0103" (id 0) (at 63.5 27.94 0)
+    (property "Reference" "#PWR016" (id 0) (at 63.5 27.94 0)
       (effects (font (size 1.27 1.27)) hide)
     )
@@
   (symbol (lib_id "power:GND") (at 63.5 43.18 0) (unit 1)
     (in_bom yes) (on_board yes) (fields_autoplaced)
-    (property "Reference" "#PWR0105" (id 0) (at 63.5 49.53 0)
+    (property "Reference" "#PWR017" (id 0) (at 63.5 49.53 0)
       (effects (font (size 1.27 1.27)) hide)
     )
@@
     (property "Reference" "LED1" (id 0) (at 72.39 31.75 0))
     (property "Value" "SK6812MINI-E" (id 1) (at 77.47 33.7693 0))
-    (property "Footprint" "LED_SK6812MINI-E" (id 2) (at 64.77 43.18 0)
+    (property "Footprint" "Skayboard:SK6812MINI-E" (id 2) (at 64.77 43.18 0)
       (effects (font (size 1.27 1.27)) (justify left top) hide)
     )
@@
   (symbol (lib_id "Device:C") (at 57.15 26.67 90) (unit 1)
     (in_bom yes) (on_board yes)
-    (property "Reference" "C1" (id 0) (at 58.42 20.32 90)
+    (property "Reference" "C7" (id 0) (at 58.42 20.32 90)
       (effects (font (size 1.27 1.27)) (justify left))
     )
@@
   (symbol (lib_id "power:GND") (at 53.34 26.67 270) (unit 1)
     (in_bom yes) (on_board yes)
-    (property "Reference" "#PWR0104" (id 0) (at 46.99 26.67 0)
+    (property "Reference" "#PWR015" (id 0) (at 46.99 26.67 0)
       (effects (font (size 1.27 1.27)) hide)
     )

Commit message: Outro - M83
Parts:
- C122: renamed from C7; footprint Capacitor_SMD:C_0402_1005Metric -> Capacitor_SMD:C_0402_1005Metric_Pad0.74x0.62mm_HandSolder
- LED116: renamed from LED1; now not fitted
