File: kicad/inc/Skey.kicad_sch (KiCad schematic)
At the start: 2 parts

Commit message: feat: finishes schematic, starts work on PCB
Parts:
- MX1: footprint (none) -> Skayboard:MX
Changed lines of the file:
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@@
       (effects (font (size 1.27 1.27)) hide)
     )
-    (property "Footprint" "" (id 2) (at 35.56 31.75 0)
+    (property "Footprint" "Skayboard:MX" (id 2) (at 29.21 36.83 0)
       (effects (font (size 1.27 1.27)) hide)
     )

Commit message: Outro - M83
Parts:
- D29: renamed from D1; footprint Diode_SMD:D_SOD-323 -> Diode_SMD:D_SOD-323_HandSoldering
- MX29: renamed from MX1; now not fitted
